Commit message: Simulation in Gazebo

File: description/robot_core.xacro (robot description, xacro)
@@ -39,8 +39,12 @@
             </geometry>
         </collision>
-        <xacro:inertial_box mass="0.5" x="0.3" y="0.3" z="0.15">
+        <xacro:inertial_box mass="6" x="0.3" y="0.3" z="0.15">
             <origin xyz="0.15 0 0.075" rpy="0 0 0"/>
         </xacro:inertial_box>
     </link>
+    <!-- set colour for Gazebo-->
+    <gazebo reference="chassis">
+        <material>Gazebo/White</material>
+    </gazebo>
     <!-- LEFT WHEEL-->
     <joint name="left_wheel_joint" type="continuous">
@@ -70,4 +74,8 @@
         </xacro:inertial_cylinder>
         </link>
+        <!-- set colour for Gazebo-->
+        <gazebo reference="left_wheel">
+            <material>Gazebo/White</material>
+        </gazebo>
     <!-- RIGHT WHEEL-->
     <joint name="right_wheel_joint" type="continuous">
@@ -97,4 +105,8 @@
         </xacro:inertial_cylinder>
         </link>
+        <!-- set colour for Gazebo-->
+        <gazebo reference="right_wheel">
+            <material>Gazebo/Blue</material>
+        </gazebo>
     <!-- CASTER WHEEL LINK-->
         <joint name="caster_wheel_joint" type="fixed">
@@ -120,3 +132,9 @@
         </xacro:inertial_sphere>
         </link>
+        <!-- set colour for Gazebo-->
+        <gazebo reference="caster_wheel">
+            <material>Gazebo/Black</material>
+            <mu1 value="0.001"/>
+            <mu2 value="0.001"/>
+        </gazebo>
 </robot>
